File: antmicro-JOB-OCulink-expansion.kicad_pcb (KiCad board)
At the start: 2 copper layers, 2 parts, among them J1 OCuLink_x4_Amphenol_G14A42121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, J2 Plug_Samtec_ERM8_2x40_ERM8-04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

Commit message: [#74340] Component placement
Parts:
- added C1: C_10u_0402, antmicro-footprints:C_0402_1005Metric, B.Cu at (198.2, 104.2)
- added C2: C_10u_0402, antmicro-footprints:C_0402_1005Metric, B.Cu at (195.2, 107.5)
- added C3: C_10u_0402, antmicro-footprints:C_0402_1005Metric, B.Cu at (212.8, 107.3)
- added R1: R_10k_0402, antmicro-footprints:R_0402_1005Metric, B.Cu at (198.2, 103.2)
- J1, J2: moved to B.Cu
- moved J2 57.9 mm to (207.1, 83.6), turned to -90 degrees
- moved J1 24.3 mm to (204.0, 110.0), turned to 180 degrees
Connections:
- J1 pad A1: unconnected-(J1-V_{ACT}_RX_3V3-PadA1) -> +3.3V
- J1 pad A11: Net-(J1-GND-PadA11) -> GND
- J1 pad A12: unconnected-(J1-VSP1-PadA12) -> /CLK+
- J1 pad A13: unconnected-(J1-VSP2-PadA13) -> /CLK-
- J1 pad A14: Net-(J1-GND-PadA11) -> GND
- J1 pad A17: Net-(J1-GND-PadA11) -> GND
- J1 pad A2: Net-(J1-GND-PadA11) -> GND
- J1 pad A20: Net-(J1-GND-PadA11) -> GND
- J1 pad A21: Net-(J1-5V-PadA21) -> +5V
- J1 pad A3: unconnected-(J1-PER0+-PadA3) -> /PER0+
- J1 pad A4: unconnected-(J1-PER0--PadA4) -> /PER0-
- J1 pad A5: Net-(J1-GND-PadA11) -> GND
- J1 pad A6: unconnected-(J1-PER1+-PadA6) -> /PER1+
- J1 pad A7: unconnected-(J1-PER1--PadA7) -> /PER1-
- J1 pad A8: Net-(J1-GND-PadA11) -> GND
- J1 pad B1: Net-(J1-5V-PadA21) -> +5V
- J1 pad B10: unconnected-(J1-SDA-PadB10) -> /SYS_SDA
- J1 pad B11: Net-(J1-GND-PadA11) -> GND
- J1 pad B12: unconnected-(J1-~{PERST}-PadB12) -> /~{RST}
- J1 pad B13: unconnected-(J1-~{CPRSNT}-PadB13) -> Net-(J1-~{CPRSNT})
- J1 pad B14: Net-(J1-GND-PadA11) -> GND
- J1 pad B17: Net-(J1-GND-PadA11) -> GND
- J1 pad B2: Net-(J1-GND-PadA11) -> GND
- J1 pad B20: Net-(J1-GND-PadA11) -> GND
- J1 pad B21: unconnected-(J1-V_{ACT}_TX_3V3-PadB21) -> +3.3V
- J1 pad B3: unconnected-(J1-PET0+-PadB3) -> /PET0+
- J1 pad B4: unconnected-(J1-PET0--PadB4) -> /PET0-
- J1 pad B5: Net-(J1-GND-PadA11) -> GND
- J1 pad B6: unconnected-(J1-PET1+-PadB6) -> /PET1+
- J1 pad B7: unconnected-(J1-PET1--PadB7) -> /PET1-
- J1 pad B8: Net-(J1-GND-PadA11) -> GND
- J1 pad B9: unconnected-(J1-SCL-PadB9) -> /SYS_SCL
- J1 pad SH: unconnected-(J1-PadSH) -> GND
- J2 pad 1: unconnected-(J2-Pad1) -> GND
- J2 pad 10: unconnected-(J2-Pad10) -> GND
- J2 pad 11: unconnected-(J2-Pad11) -> /PET0+
- J2 pad 12: unconnected-(J2-Pad12) -> /PER0-
- J2 pad 13: unconnected-(J2-Pad13) -> GND
- J2 pad 14: unconnected-(J2-Pad14) -> /PER0+
- J2 pad 15: unconnected-(J2-Pad15) -> /CLK-
- J2 pad 16: unconnected-(J2-Pad16) -> GND
- J2 pad 17: unconnected-(J2-Pad17) -> /CLK+
- J2 pad 19: unconnected-(J2-Pad19) -> GND
- J2 pad 2: unconnected-(J2-Pad2) -> GND
- J2 pad 22: unconnected-(J2-Pad22) -> GND
- J2 pad 25: unconnected-(J2-Pad25) -> GND
- J2 pad 27: unconnected-(J2-Pad27) -> /~{RST}
- J2 pad 28: unconnected-(J2-Pad28) -> GND
- J2 pad 3: unconnected-(J2-Pad3) -> /PET1-
- J2 pad 37: unconnected-(J2-Pad37) -> GND
- J2 pad 38: unconnected-(J2-Pad38) -> GND
- J2 pad 4: unconnected-(J2-Pad4) -> GND
- J2 pad 49: unconnected-(J2-Pad49) -> GND
- J2 pad 5: unconnected-(J2-Pad5) -> /PET1+
- J2 pad 50: unconnected-(J2-Pad50) -> GND
- J2 pad 6: unconnected-(J2-Pad6) -> /PER1-
- J2 pad 61: unconnected-(J2-Pad61) -> GND
- J2 pad 62: unconnected-(J2-Pad62) -> GND
- J2 pad 63: unconnected-(J2-Pad63) -> /SYS_SDA
- J2 pad 65: unconnected-(J2-Pad65) -> /SYS_SCL
- J2 pad 67: unconnected-(J2-Pad67) -> +3.3V
- J2 pad 69: unconnected-(J2-Pad69) -> +3.3V
- J2 pad 7: unconnected-(J2-Pad7) -> GND
- J2 pad 71: unconnected-(J2-Pad71) -> GND
- J2 pad 72: unconnected-(J2-Pad72) -> GND
- J2 pad 75: unconnected-(J2-Pad75) -> GND
- J2 pad 76: unconnected-(J2-Pad76) -> GND
- J2 pad 77: unconnected-(J2-Pad77) -> +5V
- J2 pad 79: unconnected-(J2-Pad79) -> +5V
- J2 pad 8: unconnected-(J2-Pad8) -> /PER1+
- J2 pad 9: unconnected-(J2-Pad9) -> /PET0-
Other:
- board outline added: 20 x 60 mm

Commit message: [#74340] Routing
Parts:
- moved J1 52.4 mm to (204.1, 57.6), turned to 0 degrees
- moved C2 51.5 mm to (212.8, 59.1)
- moved C3 50.1 mm to (195.3, 60.4), turned to 90 degrees
- moved C1 42.3 mm to (209.2, 63.4), turned to 180 degrees
- moved R1 41.1 mm to (211.7, 64.4), turned to 0 degrees
Routing:
- net +3.3V: track 0.00 -> 90.4 mm, vias 0 -> 4
- net GND: track 0.00 -> 50.7 mm, vias 0 -> 45
- net /SYS_SCL: track 0.00 -> 36.8 mm, vias 0 -> 2
- net /SYS_SDA: track 0.00 -> 35.7 mm, vias 0 -> 2
- net /PER0+: track 0.00 -> 33.0 mm, vias 0 -> 2
- net /PER0-: track 0.00 -> 30.4 mm, vias 0 -> 2
- net /PER1+: track 0.00 -> 23.7 mm, vias 0 -> 2
- net /PER1-: track 0.00 -> 21.3 mm, vias 0 -> 2
- net /CLK+: track 0.00 -> 19.8 mm, vias 0 -> 2
- net /~{RST}: track 0.00 -> 19.1 mm, vias 0 -> 2
- net /CLK-: track 0.00 -> 18.9 mm, vias 0 -> 2
- net /PET0+: track 0.00 -> 13.1 mm
- net /PET0-: track 0.00 -> 12.3 mm
- net /PET1+: track 0.00 -> 9.95 mm
- net /PET1-: track 0.00 -> 9.25 mm
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- added copper zone on B.Cu, net +5V
- added copper zone on In1.Cu, net GND
- added copper zone on In2.Cu, net GND
Other:
- copper layers 2 -> 4

Commit message: [#74340] Apply Fixes
Routing:
- net +5V: track 3.68 -> 0.00 mm
- net GND: track 50.7 -> 52.2 mm
- net /PER0-: track 30.4 -> 31.5 mm
- net /PER1-: track 21.3 -> 21.9 mm

Commit message: [#74340] Add stiching vias
Routing:
- net GND: track 52.2 -> 53.2 mm, vias 45 -> 48
Changed lines of the file:
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@@
+	)
+	(via
+		(at 211.399 70.566)
+		(size 0.6)
+		(drill 0.3)
+		(layers "F.Cu" "B.Cu")
+		(net 51)
+	)
+	(via
+		(at 201.62 71.201)
+		(size 0.45)
+		(drill 0.2)
+		(layers "F.Cu" "B.Cu")
+		(net 51)
 	)
 	(via
@@
 	)
 	(via
-		(at 203.779 61.041)
+		(at 204.033 60.914)
 		(size 0.6)
 		(drill 0.3)
@@
 	)
 	(via
-		(at 206.827 61.041)
+		(at 206.192 60.914)
 		(size 0.6)
 		(drill 0.3)
@@
 	)
 	(via
-		(at 210.129 68.626003)
+		(at 210.233333 69.000013)
 		(size 0.6)
 		(drill 0.3)
@@
 	)
 	(via
-		(at 210.256 71.035997)
+		(at 210.383 71.328)
 		(size 0.6)
 		(drill 0.3)
@@
 	)
 	(via
+		(at 200.35 72.471)
+		(size 0.45)
+		(drill 0.2)
+		(layers "F.Cu" "B.Cu")
+		(net 51)
+	)
+	(via
 		(at 206.446 75.138)
 		(size 0.6)
@@
 	)
 	(via
-		(at 210.256 73.436006)
+		(at 210.383 73.371003)
 		(size 0.6)
 		(drill 0.3)
@@
 	)
 	(segment
+		(start 204.033 60.914)
+		(end 203.803 61.144)
+		(width 0.25)
+		(layer "B.Cu")
+		(net 51)
+	)
+	(segment
 		(start 212.385 56.82)
 		(end 212.415 56.85)
@@
 	)
 	(segment
-		(start 209.957003 68.798)
-		(end 208.997 68.798)
-		(width 0.25)
-		(layer "B.Cu")
-		(net 51)
-	)
-	(segment
 		(start 202.303 61.089)
 		(end 202.255 61.041)
@@
 	)
 	(segment
-		(start 203.803 61.065)
-		(end 203.779 61.041)
-		(width 0.25)
-		(layer "B.Cu")
-		(net 51)
-	)
-	(segment
 		(start 210.963 56.82)
 		(end 212.385 56.82)
@@
 	)
 	(segment
+		(start 210.253 71.198)
+		(end 208.997 71.198)
+		(width 0.25)
+		(layer "B.Cu")
+		(net 51)
+	)
+	(segment
+		(start 210.03132 68.798)
+		(end 208.997 68.798)
+		(width 0.25)
+		(layer "B.Cu")
+		(net 51)
+	)
+	(segment
 		(start 210.34 78.397)
 		(end 210.383 78.44)
@@
 	)
 	(segment
-		(start 210.129 68.626003)
-		(end 209.957003 68.798)
-		(width 0.25)
-		(layer "B.Cu")
-		(net 51)
-	)
-	(segment
 		(start 199.303 61.93)
 		(end 199.303 61.199)
@@
 	)
 	(segment
-		(start 208.997 71.198)
-		(end 210.093997 71.198)
-		(width 0.25)
-		(layer "B.Cu")
-		(net 51)
-	)
-	(segment
 		(start 210.353 91.999)
 		(end 210.383 92.029)
@@
 	)
 	(segment
+		(start 206.192 60.914)
+		(end 206.199408 60.914)
+		(width 0.25)
+		(layer "B.Cu")
+		(net 51)
+	)
+	(segment
+		(start 206.803 61.517592)
+		(end 206.803 61.93)
+		(width 0.25)
+		(layer "B.Cu")
+		(net 51)
+	)
+	(segment
 		(start 200.803 61.199613)
 		(end 200.846597 61.156016)
@@
 	)
 	(segment
-		(start 210.093006 73.599)
-		(end 208.997 73.599)
+		(start 203.803 61.144)
+		(end 203.803 61.93)
+		(width 0.25)
+		(layer "B.Cu")
+		(net 51)
+	)
+	(segment
+		(start 206.199408 60.914)
+		(end 206.803 61.517592)
 		(width 0.25)
 		(layer "B.Cu")
@@
 	)
 	(segment
-		(start 206.803 61.065)
-		(end 206.827 61.041)
-		(width 0.25)
-		(layer "B.Cu")
-		(net 51)
-	)
-	(segment
 		(start 205.198 91.999)
 		(end 206.543 91.999)
@@
 	)
 	(segment
-		(start 206.803 61.93)
-		(end 206.803 61.065)
-		(width 0.25)
-		(layer "B.Cu")
-		(net 51)
-	)
-	(segment
-		(start 210.093997 71.198)
-		(end 210.256 71.035997)
-		(width 0.25)
-		(layer "B.Cu")
-		(net 51)
-	)
-	(segment
 		(start 208.997 97.598)
 		(end 210.364 97.598)
@@
 	)
 	(segment
+		(start 210.383 73.371003)
+		(end 210.155003 73.599)
+		(width 0.25)
+		(layer "B.Cu")
+		(net 51)
+	)
+	(segment
 		(start 204.303 59.74)
 		(end 204.303 58.955432)
@@
 	)
 	(segment
+		(start 210.383 71.328)
+		(end 210.253 71.198)
+		(width 0.25)
+		(layer "B.Cu")
+		(net 51)
+	)
+	(segment
 		(start 197.175 62.819)
 		(end 197.143 62.787)
@@
 	)
 	(segment
-		(start 203.803 61.93)
-		(end 203.803 61.065)
-		(width 0.25)
-		(layer "B.Cu")
-		(net 51)
-	)
-	(segment
 		(start 210.633 87.199)
 		(end 210.637 87.203)
@@
 	)
 	(segment
+		(start 210.155003 73.599)
+		(end 208.997 73.599)
+		(width 0.25)
+		(layer "B.Cu")
+		(net 51)
+	)
+	(segment
 		(start 202.803 60.465909)
 		(end 202.88073 60.543639)
@@
 	)
 	(segment
-		(start 210.256 73.436006)
-		(end 210.093006 73.599)
-		(width 0.25)
-		(layer "B.Cu")
-		(net 51)
-	)
-	(segment
 		(start 205.303 61.93)
 		(end 205.303 62.385)
@@
 		(width 0.25)
 		(layer "B.Cu")
+		(net 51)
+	)
+	(segment
+		(start 210.233333 69.000013)
+		(end 210.03132 68.798)
+		(width 0.25)
+		(layer "B.Cu")

Commit message: [#74340] Add Logo
Parts:
- added REF**: OSHW-Logo_5.7x6mm_Mask, antmicro-footprints:OSHW-Logo_5.7x6mm_Mask, F.Cu at (197.8, 103.0)
- added REF**: OSHW-Logo_5.7x6mm_Copper, antmicro-footprints:OSHW-Logo_5.7x6mm_Copper, F.Cu at (197.8, 103.0)
- added REF**: LOGO, antmicro-footprints:antmicro-logo_scaled_12mm, F.Cu at (201.4, 110.4)
Other:
- board text added: "JOB OCuLink Exapnsion Rev. ${REVISION} 3/2025"

Commit message: [#74340] Add PCB SHA
Parts:
- moved REF** 1.15 mm to (201.5, 109.3)
- moved REF** 1.15 mm to (197.9, 101.8) (x2)
Other:
- board text added: "PCB SHA ########"
Changed lines of the file:
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@@
 	(footprint "antmicro-footprints:OSHW-Logo_5.7x6mm_Mask"
 		(layer "F.Cu")
-		(at 197.81 102.951)
+		(at 197.937 101.808)
 		(descr "Open Source Hardware Logo")
 		(tags "Logo OSHW")
@@
 	(footprint "antmicro-footprints:OSHW-Logo_5.7x6mm_Copper"
 		(layer "F.Cu")
-		(at 197.81 102.951)
+		(at 197.937 101.808)
 		(descr "Open Source Hardware Logo")
 		(tags "Logo OSHW")
@@
 	(footprint "antmicro-footprints:antmicro-logo_scaled_12mm"
 		(layer "F.Cu")
-		(at 201.366 110.444)
+		(at 201.493 109.301)
 		(property "Reference" "REF**"
 			(at 0 -1.5 0)
@@
 	)
 	(gr_text "JOB OCuLink Exapnsion\nRev. ${REVISION}   3/2025"
-		(at 199.08 112.095 0)
+		(at 199.207 110.952 0)
 		(layer "F.Cu")
 		(effects
@@
 		)
 	)
+	(gr_text "PCB SHA ########"
+		(at 208.224 112.476 0)
+		(layer "B.SilkS")
+		(effects
+			(font
+				(size 0.65 0.65)
+				(thickness 0.15)
+			)
+			(justify mirror)
+		)
+	)
 	(gr_text "JOB OCuLink Exapnsion\nRev. ${REVISION}   3/2025"
-		(at 199.08 112.095 0)
+		(at 199.207 110.952 0)
 		(layer "F.Mask")
 		(effects
