File: antmicro-JOB-OCulink-expansion.kicad_sch (KiCad schematic)
At the start: 2 parts, among them J1 OCuLink_x4_Amphenol_G14A42121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, J2 Plug_Samtec_ERM8_2x40_ERM8-04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

Commit message: [#74340] Finished schematic
Parts:
- added C1, C2, C3: C_10u_0402, antmicro-footprints:C_0402_1005Metric, symbol antmicroCapacitors0402:C_10u_0402
- added R1: R_10k_0402, antmicro-footprints:R_0402_1005Metric, symbol antmicroResistors0402:R_10k_0402
Connections:
- net +3.3V: now also J1.A1 (V_{ACT}_RX_3V3), J1.B21 (V_{ACT}_TX_3V3), C1.2, C3.2, R1.2
- net +5V: now also J1.A21 (5V), J1.B1 (5V), C2.2
- net CLK+: now also J1.A12 (VSP1)
- net CLK-: now also J1.A13 (VSP2)
- net GND: now also J1.SH, C1.1, C2.1, C3.1
- net PER0+: now also J1.A3 (PER0+)
- net PER0-: now also J1.A4 (PER0-)
- net PER1+: now also J1.A6 (PER1+)
- net PER1-: now also J1.A7 (PER1-)
- net PET0+: now also J1.B3 (PET0+)
- net PET0-: now also J1.B4 (PET0-)
- net PET1+: now also J1.B6 (PET1+)
- net PET1-: now also J1.B7 (PET1-)
- net SYS_SCL: now also J1.B9 (SCL)
- net SYS_SDA: now also J1.B10 (SDA)
- net ~{RST}: now reaches J1.B12 (~{PERST})
- net ~{RST}: now also J2.27
- net at J1.B13 (~{CPRSNT}): now also R1.1
- no-connect marks 0 -> 51
Other:
- moved on the sheet: J1

Commit message: [#74340] Add Logo
Other:
- company: (none) -> Antmicro Ltd
- title: (none) -> Jetson Orin Baseboard OCuLink Exapnsion

Commit message: [#74340] Schematic fixes
Parts:
- removed R1: R_10k_0402, antmicro-footprints:R_0402_1005Metric, symbol antmicroResistors0402:R_10k_0402
- added C4: C_10u_0402, antmicro-footprints:C_0402_1005Metric, symbol antmicroCapacitors0402:C_10u_0402
- added C5, C6: C_100n_0402, antmicro-footprints:C_0402_1005Metric, symbol antmicroCapacitors0402:C_100n_0402
- added R1, R2: R_0R_0402, antmicro-footprints:R_0402_1005Metric, symbol antmicroResistors0402:R_0R_0402
- added R3: R_10k_0402, antmicro-footprints:R_0402_1005Metric, symbol antmicroResistors0402:R_10k_0402
- added TP1, TP10, TP2, TP3, TP4, TP5, TP6, TP7, TP8, TP9: TP_1.5mm_SMD, antmicro-footprints:TP_SMD_1.5mm, symbol antmicroTestPoints:TP_1.5mm_SMD
- added U1: MAX3373EEKA+, antmicro-footprints:SOT-23-8, symbol antmicroLogicTranslatorsLevelShifters:MAX3373EEKA+
Connections:
- net +3.3V: now also C6.2, TP8.1, U1.7 (V_{CC})
- net +5V: now also C4.2, TP9.1
- net GND: now also C4.1, C5.1, C6.1, R3.1, U1.2 (GND)
- net at J1.A10 (~{CWAKE}): now also R2.2
- net at J1.B13 (~{CPRSNT}): now also R1.2
- net JOB_GPIO07: now reaches J2.33
- net JOB_GPIO07: now also TP5.1, U1.5 (IO_V_{L}1)
- net JOB_GPIO09: now reaches J2.35
- net JOB_GPIO09: now also TP6.1, U1.4 (IO_V_{L}2)
- net +1V8: now reaches J2.73
- net +1V8: now also C5.2, TP10.1, U1.3 (V_{L})
- net CLK+ renamed PCIE_CLK+
- net CLK- renamed PCIE_CLK-
- net PER0+ renamed PCIE_RX0+
- net PER0- renamed PCIE_RX0-
- net PER1+ renamed PCIE_RX1+
- net PER1- renamed PCIE_RX1-
- net PET0+ renamed PCIE_TX0+
- net PET0- renamed PCIE_TX0-
- net PET1+ renamed PCIE_TX1+
- net PET1- renamed PCIE_TX1-
- net SYS_SCL renamed I2C_SCL
- net I2C_SCL: now also TP1.1
- net SYS_SDA renamed I2C_SDA
- net I2C_SDA: now also TP2.1
- net ~{RST} renamed ~{PCIE_RST}
- net ~{PCIE_RST}: now also TP7.1
- new net: R3.2, U1.6 (~{THREE_STATE})
- new net ~{PCIE_CPRSNT}: R1.1, TP3.1, U1.8 (IO_V_{CC}1)
- new net ~{PCIE_CWAKE}: R2.1, TP4.1, U1.1 (IO_V_{CC}2)
- no-connect marks 51 -> 47
Other:
- note added: "JOB as a ROOT Device REFCLK utilize A12+/A13"
- title: Jetson Orin Baseboard OCuLink Exapnsion -> Jetson Orin Baseboard OCuLink Expansion
- moved on the sheet: C1, C2, C3, J1, J2
